Commit message: update turtle_robot

File: turtle_brick/urdf/turtle.urdf.xacro (robot description, xacro)
@@ -36,5 +36,5 @@
         <limit effort="5.0" velocity="1.0" lower="-1.57" upper="1.57"/>
     </joint>
-    <joint name="platform_connector_to_stem" type="revolute">
+    <joint name="base_link_to_stem" type="revolute">
         <origin xyz="0 0 ${-base_link_length/2 - stem_height/2}" rpy="0 0 0"/>
         <axis xyz="0 0 1"/>
