Commit message: finished robot xacro

File: turtle_brick/urdf/_base_link.urdf.xacro (robot description, xacro)
@@ -1,8 +1,8 @@
 <robot name="base_link" xmlns:xacro="http://www.ros.org/wiki/xacro">
     <xacro:property name="yaml_file" value="$(find turtle_brick)/config/turtle.yaml" />
-    <xacro:property name="props" value="${xacro.load_yaml(${yaml_file})['/**']['ros__parameters']}" />
-    <xacro:property name="base_link_length"  value="float(props['base_link_length'])" />
-    <!-- <xacro:macro name="base_link" params="base_link_length">
-        <link name="base_link">
+    <xacro:property name="props" value="${xacro.load_yaml(yaml_file)}" />
+    <xacro:property name="base_link_length"  value="${props['base_link_length']}" />
+    <xacro:macro name="base_link" params="name">
+        <link name="${name}">
             <visual>
                 <geometry>
@@ -10,24 +10,8 @@
                 </geometry>
                 <material name="base_link_color">
-                    <color rgba="0.5 0.5 0.0 1.0"/>
+                    <color rgba="1.0 1.0 0.0 1.0"/>
                 </material>
             </visual>
         </link>
-    </xacro:macro> -->
-    <!-- <xacro:base_link base_link_length="${base_link_length}"/> -->
-    <link name="base_link">
-        <visual>
-            <geometry>
-                <box size="${base_link_length} ${base_link_length} ${base_link_length}"/>
-            </geometry>
-            <material name="base_link_color">
-                <color rgba="0.5 0.5 0.0 1.0"/>
-            </material>
-        </visual>
-    </link>
-    <link name="world"/>
-    <joint name="w2b" type="fixed">
-        <parent link="world"/>
-        <child link="base_link"/>
-    </joint>
+    </xacro:macro>
 </robot>

File: turtle_brick/urdf/turtle.urdf.xacro (robot description, xacro)
@@ -1,8 +1,52 @@
 <?xml version="1.0"?>
 <robot name="turtle" xmlns:xacro="http://www.ros.org/wiki/xacro">
+    <!-- Load the turtle.yaml file -->
     <xacro:property name="yaml_file" value="$(find turtle_brick)/config/turtle.yaml" />
     <xacro:property name="props" value="${xacro.load_yaml(yaml_file)}" />
+    <!-- Load xacro properties -->
     <xacro:property name="base_link_length"  value="${props['base_link_length']}" />
+    <xacro:property name="platform_cylinder_height"  value="${props['platform_cylinder_height']}" />
+    <xacro:property name="platform_height"  value="${props['platform_height']}" />
+    <xacro:property name="stem_height"  value="${props['stem_height']}" />
+    <xacro:property name="wheel_radius"  value="${props['wheel_radius']}" />
+    <xacro:property name="platform_connector_height"  value="${platform_height - base_link_length/2 - platform_cylinder_height/2}" />
+    <!-- Include xacro macros -->
     <xacro:include filename="$(find turtle_brick)/urdf/_base_link.urdf.xacro" />
-    <xacro:base_link base_link_length="${base_link_length}"/>
+    <xacro:include filename="$(find turtle_brick)/urdf/_platform.urdf.xacro" />
+    <xacro:include filename="$(find turtle_brick)/urdf/_platform_connector.urdf.xacro" />
+    <xacro:include filename="$(find turtle_brick)/urdf/_stem.urdf.xacro" />
+    <xacro:include filename="$(find turtle_brick)/urdf/_wheel.urdf.xacro" />
+    <!-- Call macros to generate robot links -->
+    <xacro:base_link name="base_link"/>
+    <xacro:platform_connector name="platform_connector"/>
+    <xacro:platform name="platform"/>
+    <xacro:stem name="stem"/>
+    <xacro:wheel name="wheel"/>
+    <!-- Define joints -->
+    <joint name="base_link_to_platform_connector" type="fixed">
+        <origin xyz="0 0 ${base_link_length/2 + platform_connector_height/2}" rpy="0 0 0"/>
+        <parent link="base_link"/>
+        <child link="platform_connector"/>
+    </joint>
+    <joint name="platform_connector_to_platform" type="revolute">
+        <origin xyz="0 0 ${platform_connector_height/2 + platform_cylinder_height/2}" rpy="0 0 0"/>
+        <axis xyz="0 1 0"/>
+        <parent link="platform_connector"/>
+        <child link="platform"/>
+        <limit effort="5.0" velocity="1.0" lower="-1.57" upper="1.57"/>
+    </joint>
+    <joint name="platform_connector_to_stem" type="revolute">
+        <origin xyz="0 0 ${-base_link_length/2 - stem_height/2}" rpy="0 0 0"/>
+        <axis xyz="0 0 1"/>
+        <parent link="base_link"/>
+        <child link="stem"/>
+        <limit effort="5.0" velocity="1.0" lower="-1.57" upper="1.57"/>
+    </joint>
+    <joint name="stem_to_wheel" type="revolute">
+        <origin xyz="0 0 ${-stem_height/2 - wheel_radius}" rpy="0 0 0"/>
+        <axis xyz="0 1 0"/>
+        <parent link="stem"/>
+        <child link="wheel"/>
+        <limit effort="5.0" velocity="1.0" lower="-1.57" upper="1.57"/>
+    </joint>
 </robot>

Commit message: goal_pose test passed

File: turtle_brick/urdf/_base_link.urdf.xacro (robot description, xacro)
@@ -1,5 +1,5 @@
 <robot name="base_link" xmlns:xacro="http://www.ros.org/wiki/xacro">
     <xacro:property name="yaml_file" value="$(find turtle_brick)/config/turtle.yaml" />
-    <xacro:property name="props" value="${xacro.load_yaml(yaml_file)}" />
+    <xacro:property name="props" value="${xacro.load_yaml(yaml_file)['/**']['ros__parameters']}" />
     <xacro:property name="base_link_length"  value="${props['base_link_length']}" />
     <xacro:macro name="base_link" params="name">

File: turtle_brick/urdf/_platform.urdf.xacro (robot description, xacro)
@@ -1,5 +1,5 @@
 <robot name="base_link" xmlns:xacro="http://www.ros.org/wiki/xacro">
     <xacro:property name="yaml_file" value="$(find turtle_brick)/config/turtle.yaml" />
-    <xacro:property name="props" value="${xacro.load_yaml(yaml_file)}" />
+    <xacro:property name="props" value="${xacro.load_yaml(yaml_file)['/**']['ros__parameters']}" />
     <xacro:property name="platform_cylinder_radius"  value="${props['platform_cylinder_radius']}" />
     <xacro:property name="platform_cylinder_height"  value="${props['platform_cylinder_height']}" />

File: turtle_brick/urdf/_platform_connector.urdf.xacro (robot description, xacro)
@@ -1,5 +1,5 @@
 <robot name="base_link" xmlns:xacro="http://www.ros.org/wiki/xacro">
     <xacro:property name="yaml_file" value="$(find turtle_brick)/config/turtle.yaml" />
-    <xacro:property name="props" value="${xacro.load_yaml(yaml_file)}" />
+    <xacro:property name="props" value="${xacro.load_yaml(yaml_file)['/**']['ros__parameters']}" />
     <xacro:property name="base_link_length"  value="${props['base_link_length']}" />
     <xacro:property name="platform_cylinder_radius"  value="${props['platform_cylinder_radius']}" />

File: turtle_brick/urdf/_stem.urdf.xacro (robot description, xacro)
@@ -1,5 +1,5 @@
 <robot name="base_link" xmlns:xacro="http://www.ros.org/wiki/xacro">
     <xacro:property name="yaml_file" value="$(find turtle_brick)/config/turtle.yaml" />
-    <xacro:property name="props" value="${xacro.load_yaml(yaml_file)}" />
+    <xacro:property name="props" value="${xacro.load_yaml(yaml_file)['/**']['ros__parameters']}" />
     <xacro:property name="stem_radius"  value="${props['stem_radius']}" />
     <xacro:property name="stem_height"  value="${props['stem_height']}" />

File: turtle_brick/urdf/_wheel.urdf.xacro (robot description, xacro)
@@ -1,5 +1,5 @@
 <robot name="base_link" xmlns:xacro="http://www.ros.org/wiki/xacro">
     <xacro:property name="yaml_file" value="$(find turtle_brick)/config/turtle.yaml" />
-    <xacro:property name="props" value="${xacro.load_yaml(yaml_file)}" />
+    <xacro:property name="props" value="${xacro.load_yaml(yaml_file)['/**']['ros__parameters']}" />
     <xacro:property name="wheel_radius"  value="${props['wheel_radius']}" />
     <xacro:property name="wheel_height"  value="${props['wheel_height']}" />

File: turtle_brick/urdf/turtle.urdf.xacro (robot description, xacro)
@@ -3,5 +3,5 @@
     <!-- Load the turtle.yaml file -->
     <xacro:property name="yaml_file" value="$(find turtle_brick)/config/turtle.yaml" />
-    <xacro:property name="props" value="${xacro.load_yaml(yaml_file)}" />
+    <xacro:property name="props" value="${xacro.load_yaml(yaml_file)['/**']['ros__parameters']}" />
     <!-- Load xacro properties -->
     <xacro:property name="base_link_length"  value="${props['base_link_length']}" />
@@ -23,4 +23,5 @@
     <xacro:stem name="stem"/>
     <xacro:wheel name="wheel"/>
+    <link name="base_footprint"/>
     <!-- Define joints -->
     <joint name="base_link_to_platform_connector" type="fixed">
@@ -50,3 +51,8 @@
         <limit effort="5.0" velocity="1.0" lower="-1.57" upper="1.57"/>
     </joint>
+    <joint name="base_link_to_base_footprint" type="fixed">
+        <origin xyz="0 0 -${base_link_length/2 + stem_height + wheel_radius*2}" rpy="0 0 0"/>
+        <parent link="base_link"/>
+        <child link="base_footprint"/>
+    </joint>
 </robot>
