Commit message: tilt clearing brick function testing passed

File: turtle_brick/urdf/_platform_connector.urdf.xacro (robot description, xacro)
@@ -8,6 +8,8 @@
     <xacro:property name="platform_connector_radius_ratio"  value="${props['platform_connector_radius_ratio']}" />
     <xacro:property name="platform_height"  value="${props['platform_height']}" />
+    <xacro:property name="stem_height"  value="${props['stem_height']}" />
+    <xacro:property name="wheel_radius"  value="${props['wheel_radius']}" />
     <xacro:property name="radius"  value="${platform_cylinder_radius*platform_connector_radius_ratio}" />
-    <xacro:property name="length"  value="${platform_height - base_link_length/2 - platform_cylinder_height/2}" />
+    <xacro:property name="length"  value="${platform_height - platform_cylinder_height - base_link_length - stem_height - wheel_radius*2}" />
     <xacro:macro name="platform_connector" params="name">
         <link name="${name}">

File: turtle_brick/urdf/turtle.urdf.xacro (robot description, xacro)
@@ -10,5 +10,5 @@
     <xacro:property name="stem_height"  value="${props['stem_height']}" />
     <xacro:property name="wheel_radius"  value="${props['wheel_radius']}" />
-    <xacro:property name="platform_connector_height"  value="${platform_height - base_link_length/2 - platform_cylinder_height/2}" />
+    <xacro:property name="platform_connector_height"  value="${platform_height - platform_cylinder_height - base_link_length - stem_height - wheel_radius*2}" />
     <!-- Include xacro macros -->
     <xacro:include filename="$(find turtle_brick)/urdf/_base_link.urdf.xacro" />
